Commit message: maybe can use

File: swerve_drive_description/urdf/swerve_drive.gazebo.xacro (robot description, xacro)
@@ -14,5 +14,5 @@
     </plugin>
   </gazebo>
-  <gazebo reference="base_link">
+  <gazebo reference="base_link_m">
     <mu1>0.2</mu1>
     <mu2>0.2</mu2>

File: swerve_drive_description/urdf/swerve_drive.urdf (robot description, URDF)
Before this commit: robot swerve_drive, 9 links, 8 joints
Links:
- removed link base_link
- added link base_link_m, mass 9.9142; collision mesh filename=package://swerve_drive_description/meshes/base_link.STL; visual mesh filename=package://swerve_drive_description/meshes/base_link.STL
Joints:
- joint lf_swerve_joint: parent base_link -> base_link_m
- joint lr_swerve_joint: parent base_link -> base_link_m
- joint rf_swerve_joint: parent base_link -> base_link_m
- joint rr_swerve_joint: parent base_link -> base_link_m

File: swerve_drive_description/urdf/swerve_drive.xacro (robot description, xacro)
@@ -3,14 +3,32 @@
   <xacro:include filename="$(find swerve_drive_description)/urdf/wheel.xacro" />
   <xacro:include filename="$(find swerve_drive_description)/urdf/swerve_drive.gazebo.xacro" />
-  <link name="base_footprint"/>
+  <xacro:include filename="$(find hector_sensors_description)/urdf/hokuyo_utm30lx.urdf.xacro" />
+  <!-- Hokuyo descripitions-->
+    <xacro:hokuyo_utm30lx name="front_lidar" parent="base_link_m" ros_topic="laser_front"
+                          update_rate="30" ray_count="270"
+                          min_angle="-135" max_angle="135">
+      <origin xyz="0.38516904756 0.28066904756 0.11" rpy="${M_PI} 0 ${M_PI/4}" />
+    </xacro:hokuyo_utm30lx>
+    <xacro:hokuyo_utm30lx name="back_lidar" parent="base_link_m" ros_topic="laser_back"
+                          update_rate="30" ray_count="270"
+                          min_angle="-135" max_angle="135">
+      <origin xyz="-0.38616904756 -0.28066904756 0.11" rpy="${M_PI} 0 ${M_PI/4+M_PI}" />
+    </xacro:hokuyo_utm30lx>
+  <!-- <link name="odom"/>
   <joint name="base_joint " type="fixed">
     <origin
       xyz="0 0 0.0485"
       rpy="0 0 0" />
-    <parent link="base_footprint"/>
+    <parent link="odom"/>
     <child link="base_link"/>
-  </joint>
+  </joint> -->
+  <link name="odom">
+   </link>
+  <joint name="dummy_joint" type="fixed">
+     <parent link="odom"/>
+     <child link="base_link_m"/>
+   </joint>
   <link
-    name="base_link">
+    name="base_link_m">
     <inertial>
       <origin
@@ -51,14 +69,14 @@
     </collision>
   </link>
-  <xacro:swerve_wheel side="lf_"  parent="base_link">
+  <xacro:swerve_wheel side="lf_"  parent="base_link_m">
     <origin xyz="0.24858 0.17929 0.096509" rpy="0 0 0" />
   </xacro:swerve_wheel>
-  <xacro:swerve_wheel side="rf_"  parent="base_link">
+  <xacro:swerve_wheel side="rf_"  parent="base_link_m">
     <origin xyz="0.24858 -0.18071 0.096509" rpy="0 0 0" />
   </xacro:swerve_wheel>
-  <xacro:swerve_wheel side="rr_"  parent="base_link">
+  <xacro:swerve_wheel side="rr_"  parent="base_link_m">
     <origin xyz="-0.28642 -0.18071 0.096509" rpy="0 0 0" />
   </xacro:swerve_wheel>
-  <xacro:swerve_wheel side="lr_"  parent="base_link">
+  <xacro:swerve_wheel side="lr_"  parent="base_link_m">
     <origin xyz="-0.28642 0.17929 0.096509" rpy="0 0 0" />
   </xacro:swerve_wheel>
